File: BottomBoardCam/BottomBoardCam.kicad_pcb (KiCad board)
At the start: 2 copper layers, 15 parts, among them J1 Conn_01x02_Pin, J2 43650-0528, Q1 BC817, Q2 BC817, Q3 BC817, U1 ESP32-CAM, U3 FT232RL

Commit message: svocanboard
Routing:
- net AN_IN_1: track 4.71 -> 31.9 mm
- net GND: track 80.3 -> 67.2 mm
- added copper zone on B.Cu, net (none)
- added copper zone on F.Cu, net (none)
Changed lines of the file:
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@@
-	)
-	(segment
-		(start 151.055 91.61866)
-		(end 151.055 85.555)
-		(width 0.2)
-		(layer "F.Cu")
-		(net 1)
 	)
 	(segment
@@
 	)
 	(segment
-		(start 150.18516 92.4885)
-		(end 151.055 91.61866)
-		(width 0.2)
-		(layer "F.Cu")
-		(net 1)
-	)
-	(segment
 		(start 148.76 78.26)
 		(end 145.14 78.26)
@@
 	)
 	(segment
-		(start 146.5 96)
-		(end 146.5 95)
-		(width 0.2)
-		(layer "F.Cu")
-		(net 1)
-	)
-	(segment
-		(start 149.0115 92.4885)
-		(end 150.18516 92.4885)
-		(width 0.2)
-		(layer "F.Cu")
-		(net 1)
-	)
-	(segment
 		(start 154.5 94.554468)
 		(end 154.5 85.5)
@@
 		(start 146.5 96)
 		(end 149 96)
-		(width 0.2)
-		(layer "F.Cu")
-		(net 1)
-	)
-	(segment
-		(start 146.5 95)
-		(end 149.0115 92.4885)
 		(width 0.2)
 		(layer "F.Cu")
@@
 	)
 	(segment
+		(start 148 81.95)
+		(end 147.5 81.45)
+		(width 0.2)
+		(layer "F.Cu")
+		(net 17)
+	)
+	(segment
+		(start 148 85)
+		(end 148 81.95)
+		(width 0.2)
+		(layer "F.Cu")
+		(net 17)
+	)
+	(segment
+		(start 147.5 94.00134)
+		(end 149.00134 92.5)
+		(width 0.2)
+		(layer "F.Cu")
+		(net 17)
+	)
+	(segment
+		(start 147.5 81)
+		(end 147.3 80.8)
+		(width 0.2)
+		(layer "F.Cu")
+		(net 17)
+	)
+	(segment
 		(start 149 97.825)
 		(end 146.575 97.825)
@@
 	)
 	(segment
+		(start 151 92.5)
+		(end 151 88)
+		(width 0.2)
+		(layer "F.Cu")
+		(net 17)
+	)
+	(segment
+		(start 147.5 81.45)
+		(end 147.5 81)
+		(width 0.2)
+		(layer "F.Cu")
+		(net 17)
+	)
+	(segment
+		(start 151 88)
+		(end 148 85)
+		(width 0.2)
+		(layer "F.Cu")
+		(net 17)
+	)
+	(segment
 		(start 146.575 97.825)
 		(end 146.5 97.9)
@@
 	)
 	(segment
+		(start 146.5 97.9)
+		(end 145.4 97.9)
+		(width 0.2)
+		(layer "F.Cu")
+		(net 17)
+	)
+	(segment
+		(start 145.4 97.9)
+		(end 145 97.5)
+		(width 0.2)
+		(layer "F.Cu")
+		(net 17)
+	)
+	(segment
+		(start 145 97.5)
+		(end 145 95)
+		(width 0.2)
+		(layer "F.Cu")
+		(net 17)
+	)
+	(segment
+		(start 145 95)
+		(end 147.5 95)
+		(width 0.2)
+		(layer "F.Cu")
+		(net 17)
+	)
+	(segment
+		(start 149.00134 92.5)
+		(end 151 92.5)
+		(width 0.2)
+		(layer "F.Cu")
+		(net 17)
+	)
+	(segment
 		(start 149 100)
 		(end 149 97.825)
+		(width 0.2)
+		(layer "F.Cu")
+		(net 17)
+	)
+	(segment
+		(start 147.3 80.8)
+		(end 145.14 80.8)
+		(width 0.2)
+		(layer "F.Cu")
+		(net 17)
+	)
+	(segment
+		(start 147.5 95)
+		(end 147.5 94.00134)
 		(width 0.2)
 		(layer "F.Cu")
@@
 		(net 38)
 	)
+	(zone
+		(net 0)
+		(net_name "")
+		(layer "F.Cu")
+		(hatch edge 0.5)
+		(connect_pads
+			(clearance 0.02)
+		)
+		(min_thickness 0.25)
+		(filled_areas_thickness no)
+		(fill yes
+			(thermal_gap 0.5)
+			(thermal_bridge_width 0.5)
+			(island_removal_mode 1)
+			(island_area_min 10)
+		)
+		(polygon
+			(pts
+				(xy 143.5 70.5) (xy 170 70.5) (xy 170 110.5) (xy 143.5 110.5)
+			)
+		)
+	)
+	(zone
+		(net 0)
+		(net_name "")
+		(layer "B.Cu")
+		(hatch edge 0.5)
+		(priority 1)
+		(connect_pads
+			(clearance 0.02)
+		)
+		(min_thickness 0.25)
+		(filled_areas_thickness no)
+		(fill yes
+			(thermal_gap 0.5)
+			(thermal_bridge_width 0.5)
+			(island_removal_mode 1)
+			(island_area_min 10)
+		)
+		(polygon
+			(pts
+				(xy 143.5 70.5) (xy 170 70.5) (xy 170 110.5) (xy 143.5 110.5)
+			)
+		)
+	)
 	(embedded_fonts no)
