File: charger_board/charger_board/charger_board.kicad_sch (KiCad schematic)
At the start: 37 parts, among them J1 Conn_01x04_Pin, J2 Conn_01x04_Pin, Q1 Si2319CDS, Q2 BC817, U1 STM32F042K6Tx, U2 PCA82C251, U3 LM317L_SOT-89

Commit message: svocanboard
Other:
- company: (none) -> Sieben zwanzig
- title: (none) -> Placa de carregamento
- moved on the sheet: J2
Changed lines of the file:
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@@
 	(generator_version "9.0")
 	(paper "A4")
+	(title_block
+		(title "Placa de carregamento")
+		(company "Sieben zwanzig")
+		(comment 1 "Mateus Santos Dias")
+	)
 	(rectangle
 		(start 91.44 110.49)
@@
 	(text "Can bus (Conector)\n"
 		(exclude_from_sim no)
-		(at 264.922 134.62 0)
+		(at 266.192 123.19 0)
 		(effects
 			(font
@@
 	)
 	(junction
-		(at 250.19 144.78)
+		(at 251.46 133.35)
 		(diameter 0)
 		(color 0 0 0 0)
 	)
 	(junction
-		(at 250.19 137.16)
+		(at 251.46 125.73)
 		(diameter 0)
 		(color 0 0 0 0)
@@
 	(wire
 		(pts
-			(xy 250.19 139.7) (xy 252.73 139.7)
+			(xy 251.46 128.27) (xy 254 128.27)
 		)
 		(stroke
@@
 	(wire
 		(pts
-			(xy 242.57 144.78) (xy 250.19 144.78)
+			(xy 243.84 133.35) (xy 251.46 133.35)
 		)
 		(stroke
@@
 	(wire
 		(pts
-			(xy 252.73 142.24) (xy 250.19 142.24)
+			(xy 254 130.81) (xy 251.46 130.81)
 		)
 		(stroke
@@
 	(wire
 		(pts
-			(xy 250.19 137.16) (xy 250.19 139.7)
+			(xy 251.46 125.73) (xy 251.46 128.27)
 		)
 		(stroke
@@
 	(wire
 		(pts
-			(xy 250.19 142.24) (xy 250.19 144.78)
+			(xy 251.46 130.81) (xy 251.46 133.35)
 		)
 		(stroke
@@
 	(wire
 		(pts
-			(xy 252.73 137.16) (xy 250.19 137.16)
+			(xy 254 125.73) (xy 251.46 125.73)
 		)
 		(stroke
@@
 	(wire
 		(pts
-			(xy 242.57 137.16) (xy 250.19 137.16)
+			(xy 243.84 125.73) (xy 251.46 125.73)
 		)
 		(stroke
@@
 	(wire
 		(pts
-			(xy 250.19 144.78) (xy 252.73 144.78)
+			(xy 251.46 133.35) (xy 254 133.35)
 		)
 		(stroke
@@
 	(global_label "canl"
 		(shape bidirectional)
-		(at 242.57 144.78 180)
+		(at 243.84 133.35 180)
 		(fields_autoplaced yes)
 		(effects
@@
 		)
 		(property "Intersheetrefs" "${INTERSHEET_REFS}"
-			(at 234.4217 144.78 0)
+			(at 235.6917 133.35 0)
 			(effects
 				(font
@@
 	(global_label "canh"
 		(shape bidirectional)
-		(at 242.57 137.16 180)
+		(at 243.84 125.73 180)
 		(fields_autoplaced yes)
 		(effects
@@
 		)
 		(property "Intersheetrefs" "${INTERSHEET_REFS}"
-			(at 233.9379 137.16 0)
+			(at 235.2079 125.73 0)
 			(effects
 				(font
@@
 	(symbol
 		(lib_id "Connector:Conn_01x04_Pin")
-		(at 257.81 142.24 180)
+		(at 259.08 130.81 180)
 		(unit 1)
 		(exclude_from_sim no)
@@
 		(fields_autoplaced yes)
 		(property "Reference" "J2"
-			(at 259.08 139.6999 0)
+			(at 260.35 128.2699 0)
 			(effects
 				(font
@@
 		)
 		(property "Value" "Conn_01x04_Pin"
-			(at 259.08 142.2399 0)
+			(at 260.35 130.8099 0)
 			(effects
 				(font
@@
 		)
 		(property "Footprint" "Connector_PinHeader_2.54mm:PinHeader_1x04_P2.54mm_Vertical"
-			(at 257.81 142.24 0)
+			(at 259.08 130.81 0)
 			(effects
 				(font
@@
 		)
 		(property "Datasheet" "~"
-			(at 257.81 142.24 0)
+			(at 259.08 130.81 0)
 			(effects
 				(font
@@
 		)
 		(property "Description" "Generic connector, single row, 01x04, script generated"
-			(at 257.81 142.24 0)
+			(at 259.08 130.81 0)
 			(effects
 				(font

Commit message: placa bms pronta
Parts:
- removed C7: 470uF, Capacitor_THT:CP_Radial_D6.3mm_P2.50mm, symbol Device:C_Polarized
- removed D1: BAT42W-V, Diode_SMD:D_SOD-123, symbol Diode:BAT42W-V
- removed L1: 680uH, Inductor_SMD:L_Taiyo-Yuden_NR-60xx_HandSoldering, symbol Device:L
- removed Q1: Si2319CDS, Package_TO_SOT_SMD:SOT-23, symbol Transistor_FET:Si2319CDS
- removed Q2: BC817, Package_TO_SOT_SMD:SOT-23, symbol Transistor_BJT:BC817
- removed R10: 10k, Resistor_SMD:R_1206_3216Metric, symbol Device:R_US
- removed R11: 1k, Resistor_SMD:R_1206_3216Metric, symbol Device:R_US
- added D1: 1N5405, Diode_SMD:D_1206_3216Metric, symbol Diode:1N5405
- added J3, J4: Conn_01x02_Pin, Connector_PinHeader_2.54mm:PinHeader_1x02_P2.54mm_Vertical, symbol Connector:Conn_01x02_Pin
- added Q1: IRF9540N, Package_TO_SOT_SMD:TO-252-2, symbol Transistor_FET:IRF9540N
- added Q3: BC817, Package_TO_SOT_SMD:SOT-23, symbol Transistor_BJT:BC817
- added R17: 10k, Resistor_SMD:R_1206_3216Metric, symbol Device:R_US
- added R18: 1k, Resistor_SMD:R_1206_3216Metric, symbol Device:R_US
- R14: value 3k3 -> 15K
- R3: value 1k2 -> 23K
- R9: value 4k7 -> 10k
Connections:
- net +12V is gone; now on net +5V: C5.1, D2.1 (K), R12.1, U3.3 (VI)
- net GND: now also J2.1 (Pin_1), J3.1 (Pin_1), J4.1 (Pin_1), Q3.2 (E), R17.2
- net Lion_Batt: now also J2.2 (Pin_2), D1.1 (K), J4.2 (Pin_2)
- net canh: no longer J2.3 (Pin_3)
- net canl: now also J2.3 (Pin_3); no longer J2.1 (Pin_1), J2.2 (Pin_2)
- net scl_sens_pa09: now reaches U1.19 (PA9)
- net sda_sens_pa10: now reaches U1.20 (PA10)
- net +5V: now reaches R9.2
- net +5V: now also J3.2 (Pin_2), Q1.3 (S)
- net at R9.1: now also Q1.1 (G), Q3.3 (C)
- net out_enable_pa7 renamed charge_enable_pa7
- net charge_enable_pa7: now also R18.1
- net pwm_out_pa6: no longer names the net of U1.12 (PA6)
- new net: D1.2 (A), Q1.2 (D)
- new net: Q3.1 (B), R17.1, R18.2
Other:
- moved on the sheet: C1, C2, C5, C6, D2, J2, R4, R5, R6, R7, R8, U2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
